File: cad/dcc_block_detector.sch (EAGLE design)
At the start: 71 parts, among them CN1 UART_FULL_DUPLEX, CN2 UART_HALF_DUPLEX, Q1 CSTCR6M00G53Z, U2 SN74LVC1G07DCKR, U3 MCP1790-3302E/DB, U4 ADUM1201ARZ, X1 1751248

Commit message: Code working as expected. First working release.
Other:
- note added: "ALT: LP2950-33LPE3 TO92 mount as SMD"
Changed lines of the file:
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@@
 <setting verticaltext="up"/>
 </settings>
-<grid distance="50" unitdist="mil" unit="mil" style="lines" multiple="1" display="no" altdistance="0.01" altunitdist="inch" altunit="inch"/>
+<grid distance="0.1" unitdist="inch" unit="inch" style="lines" multiple="1" display="no" altdistance="0.01" altunitdist="inch" altunit="inch"/>
 <layers>
 <layer number="1" name="Top" color="4" fill="1" visible="no" active="no"/>
@@
 (C) 2015 Mikael Sundin</text>
 <text x="104.14" y="88.9" size="2.54" layer="97">Mount U2 for half-duplex uart</text>
+<text x="337.82" y="45.72" size="1.778" layer="97">ALT: LP2950-33LPE3
+TO92 mount as SMD</text>
 </plain>
 <instances>
